File: hardware/circuit/hardware.kicad_pcb (KiCad board)
At the start: 2 copper layers, 88.3 x 69.2 mm, 30 parts, among them J1 GAUGE 1, J10 7-SEG TOP, J11 7-SEG BTM, J12 INDICATORS, J2 DEBUG, J3 GAUGE 2, J4 GAUGE 3, J5 NEOPIXEL, J6 GAUGE 4, J7 GAUGE 5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

Commit message: updated readme
Parts:
- moved R4 4.39 mm to (182.6, 72.1)
- moved REF** 2.81 mm to (124.0, 83.8)
- moved REF** 2.81 mm to (204.5, 83.8)
- moved REF** 1.63 mm to (199.6, 69.1)
- moved REF** 0.36 mm to (124.0, 24.9)
- moved REF** 0.36 mm to (204.5, 24.9)
Routing:
- net Net-(J12-Pin_6): track 10.6 -> 15.3 mm
- net +3.3V: track 125.7 -> 127.5 mm
- net +5V: track 56.6 -> 58.0 mm
- net /RX: track 16.4 -> 17.1 mm
- net Net-(J4-Pin_1): track 10.9 -> 11.5 mm
- net Net-(J7-Pin_1): track 10.9 -> 11.5 mm
Other:
- board size 88.3 x 69.2 mm -> 88.3 x 66.7 mm
